Commit message: Update files for camera simulation

File: ros2_ws/src/hardware/xarm/mbot_demo/urdf/base_with_arm.urdf.xacro (robot description, xacro)
@@ -50,6 +50,6 @@
     ros2_control_plugin="$(arg ros2_control_plugin)" robot_type="$(arg robot_type)"
     load_gazebo_plugin="true" ros2_control_params="$(arg ros2_control_params)"
-    add_realsense_d435i="true"
-    add_d435i_links="false"
+    add_realsense_d435i="$(arg add_realsense_d435i)"
+    add_d435i_links="$(arg add_d435i_links)"
     add_other_geometry="$(arg add_other_geometry)"
     geometry_type="$(arg geometry_type)" geometry_mass="$(arg geometry_mass)"

File: ros2_ws/src/hardware/xarm/mbot_demo/urdf/mbot_with_xarm.urdf.xacro (robot description, xacro)
@@ -17,7 +17,7 @@
   <xacro:arg name="ros2_control_plugin" default="uf_robot_hardware/UFRobotSystemHardware"/>
   <xacro:arg name="ros2_control_params" default=""/>
-  <xacro:arg name="add_realsense_d435i" default="false"/>
+  <xacro:arg name="add_realsense_d435i" default="true"/>
   <xacro:arg name="add_d435i_links" default="true"/>
-  <xacro:arg name="use_gazebo_camera" default="false"/>
+  <xacro:arg name="use_gazebo_camera" default="true"/>
   <xacro:arg name="add_other_geometry" default="false"/>
   <xacro:arg name="geometry_type" default="box"/>

File: ros2_ws/src/hardware/xarm/xarm_description/urdf/camera/realsense_d435i.urdf.xacro (robot description, xacro)
@@ -28,5 +28,7 @@
         <parent link="${prefix}link_eef" />
         <child link="${prefix}camera_link" />
-        <origin xyz="0.06746 -0.0175 0.0237" rpy="${M_PI} ${-M_PI/2} 0" />
+        <!-- <origin xyz="0.06746 -0.0175 0.0237" rpy="${M_PI} ${-M_PI/2} 0" /> -->
+        <!-- ORIGIN CHANGED TO AVOID SEEING THE SELF-GRIPPER -->
+        <origin xyz="0.08746 -0.0175 0.0237" rpy="${M_PI} ${-M_PI/2} 0" />
       </joint>
       <joint name="${prefix}camera_depth_joint" type="fixed">

File: ros2_ws/src/hardware/xarm/xarm_description/urdf/camera/realsense_no_ir.gazebo.xacro (robot description, xacro)
@@ -21,5 +21,5 @@
         </camera>
         <always_on>1</always_on>
-        <update_rate>20</update_rate>
+        <update_rate>10</update_rate>
         <visualize>0</visualize>
       </sensor>
@@ -45,5 +45,5 @@
         </camera>
         <always_on>1</always_on>
-        <update_rate>20</update_rate>
+        <update_rate>10</update_rate>
         <visualize>1</visualize>
       </sensor>
@@ -52,12 +52,12 @@
       <plugin name="realsense_gazebo_camera" filename="librealsense_gazebo_plugin.so">
         <prefix>${prefix}camera</prefix>
-        <depthUpdateRate>20.0</depthUpdateRate>
-        <colorUpdateRate>20.0</colorUpdateRate>
+        <depthUpdateRate>10.0</depthUpdateRate>
+        <colorUpdateRate>10.0</colorUpdateRate>
         <depthTopicName>${prefix}aligned_depth_to_color/image_raw</depthTopicName>
         <depthCameraInfoTopicName>${prefix}depth/camera_info</depthCameraInfoTopicName>
         <colorTopicName>${prefix}color/image_raw</colorTopicName>
         <colorCameraInfoTopicName>${prefix}color/camera_info</colorCameraInfoTopicName>
-        <colorOpticalframeName>/camera_color_optical_frame</colorOpticalframeName>
-        <depthOpticalframeName>/camera_depth_optical_frame</depthOpticalframeName>
+        <colorOpticalframeName>${prefix}camera_color_optical_frame</colorOpticalframeName>
+        <depthOpticalframeName>${prefix}camera_depth_optical_frame</depthOpticalframeName>
         <rangeMinDepth>0.3</rangeMinDepth>
         <rangeMaxDepth>3.0</rangeMaxDepth>

File: ros2_ws/src/hardware/xarm/xarm_description/urdf/xarm_device_macro.xacro (robot description, xacro)
@@ -42,4 +42,5 @@
     mesh_suffix:='stl'
     kinematics_suffix:=''
+    is_ros2:=true
     "
     >

Commit message: new_files_a/m

File: ros2_ws/src/hardware/xarm/mbot_demo/urdf/base_with_arm.urdf.xacro (robot description, xacro)
@@ -50,6 +50,6 @@
     ros2_control_plugin="$(arg ros2_control_plugin)" robot_type="$(arg robot_type)"
     load_gazebo_plugin="true" ros2_control_params="$(arg ros2_control_params)"
-    add_realsense_d435i="true"
-    add_d435i_links="false"
+    add_realsense_d435i="$(arg add_realsense_d435i)"
+    add_d435i_links="$(arg add_d435i_links)"
     add_other_geometry="$(arg add_other_geometry)"
     geometry_type="$(arg geometry_type)" geometry_mass="$(arg geometry_mass)"

File: ros2_ws/src/hardware/xarm/xarm_description/urdf/camera/realsense_d435i.urdf.xacro (robot description, xacro)
@@ -28,5 +28,5 @@
         <parent link="${prefix}link_eef" />
         <child link="${prefix}camera_link" />
-        <origin xyz="0.06746 -0.0175 0.0237" rpy="${M_PI} ${-M_PI/2} 0" />
+        <origin xyz="0.08746 -0.0175 0.0237" rpy="${M_PI} ${-M_PI/2} 0" />
       </joint>
       <joint name="${prefix}camera_depth_joint" type="fixed">

File: ros2_ws/src/hardware/xarm/xarm_description/urdf/camera/realsense_no_ir.gazebo.xacro (robot description, xacro)
@@ -21,5 +21,5 @@
         </camera>
         <always_on>1</always_on>
-        <update_rate>20</update_rate>
+        <update_rate>10</update_rate>
         <visualize>0</visualize>
       </sensor>
@@ -45,5 +45,5 @@
         </camera>
         <always_on>1</always_on>
-        <update_rate>20</update_rate>
+        <update_rate>10</update_rate>
         <visualize>1</visualize>
       </sensor>
@@ -52,12 +52,12 @@
       <plugin name="realsense_gazebo_camera" filename="librealsense_gazebo_plugin.so">
         <prefix>${prefix}camera</prefix>
-        <depthUpdateRate>20.0</depthUpdateRate>
-        <colorUpdateRate>20.0</colorUpdateRate>
+        <depthUpdateRate>10.0</depthUpdateRate>
+        <colorUpdateRate>10.0</colorUpdateRate>
         <depthTopicName>${prefix}aligned_depth_to_color/image_raw</depthTopicName>
         <depthCameraInfoTopicName>${prefix}depth/camera_info</depthCameraInfoTopicName>
         <colorTopicName>${prefix}color/image_raw</colorTopicName>
         <colorCameraInfoTopicName>${prefix}color/camera_info</colorCameraInfoTopicName>
-        <colorOpticalframeName>/camera_color_optical_frame</colorOpticalframeName>
-        <depthOpticalframeName>/camera_depth_optical_frame</depthOpticalframeName>
+        <colorOpticalframeName>${prefix}camera_color_optical_frame</colorOpticalframeName>
+        <depthOpticalframeName>${prefix}camera_depth_optical_frame</depthOpticalframeName>
         <rangeMinDepth>0.3</rangeMinDepth>
         <rangeMaxDepth>3.0</rangeMaxDepth>

File: ros2_ws/src/hardware/xarm/xarm_description/urdf/xarm_device_macro.xacro (robot description, xacro)
@@ -42,4 +42,5 @@
     mesh_suffix:='stl'
     kinematics_suffix:=''
+    is_ros2:=true
     "
     >
