Commit message: Proyecto final Guerra Sanchez y Romero Velazquez

File: ros2_ws/src/hardware/justina_description/urdf/justina.xacro (robot description, xacro)
@@ -1,17 +1,43 @@
-<?xml version="1.0"?>
-<robot name="justina" xmlns:xacro="http://www.ros.org/wiki/xacro">
-  <xacro:include filename="$(find justina_description)/urdf/justina_base.xacro"/>
-  <!-- <xacro:include filename="$(find justina_description)/urdf/justina_upper.xacro"/> -->
-  <!-- <joint name="base_torso_joint" type="fixed"> -->
-  <!--   <origin xyz="0.0 0.0 0.375" rpy="0 0 0"/> -->
-  <!--   <parent link="body_link"/> -->
-  <!--   <child link="torso_link"/> -->
-  <!-- </joint> -->
-  <!-- <xacro:include filename="$(find xarm_description)/urdf/xarm_device.urdf.xacro"/> -->
-  <!-- <link name="justina_arm_base_link"/> -->
-  <!-- <joint name="body_arm_base_joint" type="fixed"> -->
-  <!--   <origin xyz="0 0 0.175" rpy="0 0 0"/> -->
-  <!--   <parent link="body_link"/> -->
-  <!--   <child link="justina_arm_base_link"/> -->
-  <!-- </joint> -->
+  <!-- Cámara RGB -->
+  <joint name="camera_joint" type="fixed">
+    <parent link="base_link"/>
+    <child link="camera_link"/>
+    <origin xyz="0.2 0 0.5" rpy="0 0 0"/>
+  </joint>
+  <link name="camera_link">
+    <visual>
+      <geometry>
+        <box size="0.05 0.1 0.05"/>
+      </geometry>
+      <material name="black"/>
+    </visual>
+  </link>
+  <gazebo reference="camera_link">
+    <sensor name="camera" type="camera">
+      <visualize>true</visualize>
+      <update_rate>30</update_rate>
+      <camera>
+        <horizontal_fov>1.047</horizontal_fov>
+        <image>
+          <width>640</width>
+          <height>480</height>
+          <format>R8G8B8</format>
+        </image>
+        <clip>
+          <near>0.05</near>
+          <far>30</far>
+        </clip>
+      </camera>
+      <plugin name="camera_controller" filename="libgazebo_ros_camera.so">
+        <ros>
+          <namespace>/justina</namespace>
+          <argument>camera/image_raw</argument>
+        </ros>
+        <camera_name>camera</camera_name>
+        <image_topic_name>image_raw</image_topic_name>
+        <camera_info_topic_name>camera_info</camera_info_topic_name>
+        <frame_name>camera_link</frame_name>
+      </plugin>
+    </sensor>
+  </gazebo>
 </robot>

File: ros2_ws/src/hardware/xarm/xarm_description/urdf/camera/camera.gazebo.xacro (robot description, xacro)
@@ -1,4 +1,4 @@
 <?xml version="1.0"?>
-<robot xmlns:xacro="http://ros.org/wiki/xacro">
+<robot xmlns:xacro="http://www.ros.org/wiki/xacro">
   <xacro:macro name="camera_gazebo" params="prefix">
     <link name="${prefix}link_camera">
@@ -15,5 +15,5 @@
           <sphere radius="0.02"/>
         </geometry>
-        <material name="${prefix}White" />
+        <material name="White" />
       </visual>
       <collision>
@@ -25,58 +25,31 @@
     </link>
     <joint name="${prefix}joint_camera" type="fixed">
-      <origin xyz="0.692 0.001 1.17" rpy="0 1.5708 0" />
+      <origin xyz="0.15 0 0.25" rpy="0 0 0" />
       <parent link="${prefix}link_base" />
       <child link="${prefix}link_camera" />
     </joint>
     <gazebo reference="${prefix}link_camera">
-      <material>Gazebo/Black</material>
-    </gazebo>
-    <gazebo reference="${prefix}link_camera">
-      <sensor type="camera" name="xarm_camera_node">
-        <!-- <always_on>0</always_on> -->
-        <update_rate>10.0</update_rate>
-        <camera name="head">
-          <!-- <horizontal_fov>1.3962634</horizontal_fov> -->
-          <horizontal_fov>0.9948376567</horizontal_fov>
-          <image>
+      <sensor type="camera" name="camera_sensor">
+        <update_rate>30.0</update_rate>
+        <camera name="camera">
+          <horizontal_fov>1.047</horizontal_fov>
+          <td>
             <width>640</width>
             <height>480</height>
-            <foramt>B8G8R8</foramt>
+            <format>R8G8B8</format>
           </image>
           <clip>
-            <near>0.02</near>
-            <far>300</far>
+            <near>0.05</near>
+            <far>30.0</far>
           </clip>
-          <noise>
-            <type>gaussian</type>
-            <mean>0.0</mean>
-            <stddev>0.007</stddev>
-          </noise>
         </camera>
-        <plugin name="gazebo_camera" filename="libgazebo_ros_camera.so">
-          <xacro:if value="${is_ros2}">
-            <ros>
-              <namespace>/</namespace>
-              <remapping>image_raw:=image_raw</remapping>
-              <remapping>camera_info:=camera_info</remapping>
-            </ros>
-            <camera_name>camera</camera_name>
-            <frame_name>camera_link</frame_name>
-            <hack_baseline>0.07</hack_baseline>
-          </xacro:if>
-          <xacro:unless value="${is_ros2}">
-            <alwaysOn>true</alwaysOn>
-            <updateRate>0.0</updateRate>
-            <cameraName>/camera</cameraName>
-            <imageTopicName>image_raw</imageTopicName>
-            <cameraInfoTopicName>camera_info</cameraInfoTopicName>
-            <frameName>camera_link</frameName>
-            <hackBaseline>0.07</hackBaseline>
-            <distortionK1>0.0</distortionK1>
-            <distortionK2>0.0</distortionK2>
-            <distortionK3>0.0</distortionK3>
-            <distortionT1>0.0</distortionT1>
-            <distortionT2>0.0</distortionT2>
-          </xacro:unless>
+        <plugin name="camera_controller" filename="libgazebo_ros_camera.so">
+          <ros>
+            <namespace>/</namespace>
+          </ros>
+          <camera_name>camera</camera_name>
+          <image_topic_name>image_raw</image_topic_name>
+          <camera_info_topic_name>camera_info</camera_info_topic_name>
+          <frame_name>${prefix}link_camera</frame_name>
         </plugin>
       </sensor>

File: ros2_ws/src/hardware/xarm/xarm_description/urdf/xarm_device_macro.xacro (robot description, xacro)
@@ -21,5 +21,5 @@
     add_realsense_d435i:=false
     add_d435i_links:=true
-    use_gazebo_camera:=false
+    use_gazebo_camera:=true
     add_other_geometry:=false
     geometry_type:='box'
