Commit message: Finalize sm planner demo and camera orientation

File: ros2_ws/src/hardware/xarm/xarm_description/urdf/camera/realsense_d435i.urdf.xacro (robot description, xacro)
@@ -30,5 +30,5 @@
         <!-- <origin xyz="0.06746 -0.0175 0.0237" rpy="${M_PI} ${-M_PI/2} 0" /> -->
         <!-- ORIGIN CHANGED TO AVOID SEEING THE SELF-GRIPPER -->
-        <origin xyz="0.08746 -0.0175 0.0237" rpy="${M_PI} ${-M_PI/2} 0" />
+        <origin xyz="0.08746 -0.0175 0.0237" rpy="${M_PI} 0 0" />
       </joint>
       <joint name="${prefix}camera_depth_joint" type="fixed">
